File: kicad/M17_soundcard.kicad_pcb (KiCad board)
At the start: 2 copper layers, 139 x 65 mm, 60 parts, among them IC1 74HCT04D, IC2 74HCT4017D, IC3 74HCT4017D, IC4 74HCT4046D, X1 10M_REF, X2 12MHz, X3 INP_A, X4 INP_B, X5 OUT_A, X6 OUT_B

Commit message: Changed board shape, added GND connections to USB socket, added PDF file with schematic
Parts:
- moved   61.5 mm to (144.0, 134.0)
Connections:
- CN1 pad GND1: (no net) -> GND
- CN1 pad GND2: (no net) -> GND
- CN1 pad GND3: (no net) -> GND
- CN1 pad GND4: (no net) -> GND
Routing:
- net GND: vias 112 -> 100
Other:
- outline, holes or cut-outs redrawn
- board text added: "Analog interface board Wojciech Kaczmarski SP5WWP Silvano Seva IU2KWO"
Changed lines of the file:
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@@
   (general
     (thickness 1.6)
-    (drawings 4)
-    (tracks 364)
+    (drawings 7)
+    (tracks 352)
     (zones 0)
     (modules 60)
@@
   )
   (setup
-    (last_trace_width 0.6096)
+    (last_trace_width 0.25)
     (user_trace_width 0.254)
     (user_trace_width 0.3175)
@@
     (mod_text_size 1 1)
     (mod_text_width 0.15)
-    (pad_size 1.524 1.524)
-    (pad_drill 0.762)
+    (pad_size 2 2.4)
+    (pad_drill 0)
     (pad_to_mask_clearance 0)
     (aux_axis_origin 0 0)
@@
       (drillshape 0)
       (scaleselection 1)
-      (outputdirectory "gebers/"))
+      (outputdirectory "../gebers/"))
   )
   (net 0 "")
@@
   )
   (module MountingHole:MountingHole_3.2mm_M3_ISO7380 (layer Top)
-    (at 82.5 134)
+    (at 144 134)
     (descr "Mounting Hole 3.2mm, no annular, M3, ISO7380")
     (tags "mounting hole 3.2mm no annular m3 iso7380")
@@
       (effects (font (size 1 1) (thickness 0.15)))
     )
-    (fp_text user %R (at 0.3 0) (layer F.Fab)
-      (effects (font (size 1 1) (thickness 0.15)))
-    )
     (fp_circle (center 0 0) (end 2.85 0) (layer Cmts.User) (width 0.15))
     (fp_circle (center 0 0) (end 3.1 0) (layer F.CrtYd) (width 0.05))
+    (fp_text user %R (at 0 0) (layer F.Fab)
+      (effects (font (size 1 1) (thickness 0.15)))
+    )
     (pad 1 np_thru_hole circle (at 0 0) (size 3.2 3.2) (drill 3.2) (layers *.Cu *.Mask))
   )
@@
       (effects (font (size 1 1) (thickness 0.15)))
     )
+    (fp_circle (center 0 0) (end 2.85 0) (layer Cmts.User) (width 0.15))
+    (fp_circle (center 0 0) (end 3.1 0) (layer F.CrtYd) (width 0.05))
     (fp_text user %R (at 0.3 0) (layer F.Fab)
       (effects (font (size 1 1) (thickness 0.15)))
     )
-    (fp_circle (center 0 0) (end 2.85 0) (layer Cmts.User) (width 0.15))
-    (fp_circle (center 0 0) (end 3.1 0) (layer F.CrtYd) (width 0.05))
     (pad 1 np_thru_hole circle (at 0 0) (size 3.2 3.2) (drill 3.2) (layers *.Cu *.Mask))
   )
@@
       (effects (font (size 1 1) (thickness 0.15)))
     )
+    (fp_circle (center 0 0) (end 2.85 0) (layer Cmts.User) (width 0.15))
+    (fp_circle (center 0 0) (end 3.1 0) (layer F.CrtYd) (width 0.05))
     (fp_text user %R (at 0.3 0) (layer F.Fab)
       (effects (font (size 1 1) (thickness 0.15)))
     )
-    (fp_circle (center 0 0) (end 2.85 0) (layer Cmts.User) (width 0.15))
-    (fp_circle (center 0 0) (end 3.1 0) (layer F.CrtYd) (width 0.05))
     (pad 1 np_thru_hole circle (at 0 0) (size 3.2 3.2) (drill 3.2) (layers *.Cu *.Mask))
   )
@@
     (pad "" np_thru_hole circle (at -2.2 -1) (size 1 1) (drill 1) (layers *.Cu *.Mask))
     (pad GND4 smd rect (at 4.4 2) (size 2 2.4) (layers Top F.Paste F.Mask)
-      (solder_mask_margin 0.1016))
+      (net 1 GND) (solder_mask_margin 0.1016))
     (pad GND3 smd rect (at 4.4 -3.5) (size 2 2.4) (layers Top F.Paste F.Mask)
-      (solder_mask_margin 0.1016))
+      (net 1 GND) (solder_mask_margin 0.1016))
     (pad GND1 smd rect (at -4.4 2) (size 2 2.4) (layers Top F.Paste F.Mask)
-      (solder_mask_margin 0.1016))
+      (net 1 GND) (solder_mask_margin 0.1016))
     (pad GND smd rect (at 1.6 -4.064 180) (size 0.5 2.308) (layers Top F.Paste F.Mask)
       (net 1 GND) (solder_mask_margin 0.1016))
@@
       (net 3 +5V) (solder_mask_margin 0.1016))
     (pad GND2 smd rect (at -4.4 -3.5) (size 2 2.4) (layers Top F.Paste F.Mask)
-      (solder_mask_margin 0.1016))
+      (net 1 GND) (solder_mask_margin 0.1016))
   )
   (module SOD523 (layer Top)
@@
       (net 10 N$4) (solder_mask_margin 0.1016))
   )
-  (gr_line (start 79.0011 137.5036) (end 218.0011 137.5036) (layer Edge.Cuts) (width 0.05))
+  (gr_text "Analog interface board\n\nWojciech Kaczmarski SP5WWP\nSilvano Seva IU2KWO" (at 181 131) (layer F.SilkS)
+    (effects (font (size 1 1) (thickness 0.15)) (justify left))
+  )
+  (gr_line (start 140.5 101) (end 79 101) (layer Edge.Cuts) (width 0.05))
+  (gr_line (start 140.5 137.5) (end 218 137.5) (layer Edge.Cuts) (width 0.05))
+  (gr_line (start 79 101) (end 79 72.5) (layer Edge.Cuts) (width 0.05))
+  (gr_line (start 140.5 137.5) (end 140.5 101) (layer Edge.Cuts) (width 0.05))
   (gr_line (start 218.0011 137.5036) (end 218.0011 72.5036) (layer Edge.Cuts) (width 0.05))
   (gr_line (start 218.0011 72.5036) (end 79.0011 72.5036) (layer Edge.Cuts) (width 0.05))
-  (gr_line (start 79.0011 72.5036) (end 79.0011 137.5036) (layer Edge.Cuts) (width 0.05))
   (via (at 159.893 104.034166) (size 0.8) (drill 0.4) (layers Top Bottom) (net 1))
   (via (at 159.893 102.531333) (size 0.8) (drill 0.4) (layers Top Bottom) (net 1))
@@
   (via (at 201.403599 130.429) (size 0.8) (drill 0.4) (layers Top Bottom) (net 1))
   (via (at 192.917349 130.429) (size 0.8) (drill 0.4) (layers Top Bottom) (net 1))
-  (via (at 138.1869 106.187875) (size 0.8) (drill 0.4) (layers Top Bottom) (net 1))
-  (via (at 108.4065 106.187875) (size 0.8) (drill 0.4) (layers Top Bottom) (net 1))
-  (via (at 98.4797 106.187875) (size 0.8) (drill 0.4) (layers Top Bottom) (net 1))
-  (via (at 128.2601 106.187875) (size 0.8) (drill 0.4) (layers Top Bottom) (net 1))
-  (via (at 88.5529 106.187875) (size 0.8) (drill 0.4) (layers Top Bottom) (net 1))
-  (via (at 118.3333 106.187875) (size 0.8) (drill 0.4) (layers Top Bottom) (net 1))
-  (via (at 138.1869 114.26825) (size 0.8) (drill 0.4) (layers Top Bottom) (net 1))
-  (via (at 108.4065 114.26825) (size 0.8) (drill 0.4) (layers Top Bottom) (net 1))
-  (via (at 98.4797 114.26825) (size 0.8) (drill 0.4) (layers Top Bottom) (net 1))
-  (via (at 128.2601 114.26825) (size 0.8) (drill 0.4) (layers Top Bottom) (net 1))
-  (via (at 88.5529 114.26825) (size 0.8) (drill 0.4) (layers Top Bottom) (net 1))
-  (via (at 118.3333 114.26825) (size 0.8) (drill 0.4) (layers Top Bottom) (net 1))
-  (via (at 138.1869 122.348625) (size 0.8) (drill 0.4) (layers Top Bottom) (net 1))
-  (via (at 108.4065 122.348625) (size 0.8) (drill 0.4) (layers Top Bottom) (net 1))
-  (via (at 98.4797 122.348625) (size 0.8) (drill 0.4) (layers Top Bottom) (net 1))
-  (via (at 128.2601 122.348625) (size 0.8) (drill 0.4) (layers Top Bottom) (net 1))
-  (via (at 88.5529 122.348625) (size 0.8) (drill 0.4) (layers Top Bottom) (net 1))
-  (via (at 118.3333 122.348625) (size 0.8) (drill 0.4) (layers Top Bottom) (net 1))
-  (via (at 138.1869 130.429) (size 0.8) (drill 0.4) (layers Top Bottom) (net 1))
-  (via (at 108.4065 130.429) (size 0.8) (drill 0.4) (layers Top Bottom) (net 1))
-  (via (at 98.4797 130.429) (size 0.8) (drill 0.4) (layers Top Bottom) (net 1))
-  (via (at 128.2601 130.429) (size 0.8) (drill 0.4) (layers Top Bottom) (net 1))
-  (via (at 88.5529 130.429) (size 0.8) (drill 0.4) (layers Top Bottom) (net 1))
-  (via (at 118.3333 130.429) (size 0.8) (drill 0.4) (layers Top Bottom) (net 1))
+  (via (at 142.6869 105.187875) (size 0.8) (drill 0.4) (layers Top Bottom) (net 1))
+  (via (at 128.450916 97.1075) (size 0.8) (drill 0.4) (layers Top Bottom) (net 1))
+  (via (at 114.21494 97.1075) (size 0.8) (drill 0.4) (layers Top Bottom) (net 1))
+  (via (at 145.7601 105.187875) (size 0.8) (drill 0.4) (layers Top Bottom) (net 1))
+  (via (at 99.978964 97.1075) (size 0.8) (drill 0.4) (layers Top Bottom) (net 1))
+  (via (at 135.568904 97.1075) (size 0.8) (drill 0.4) (layers Top Bottom) (net 1))
+  (via (at 142.6869 113.26825) (size 0.8) (drill 0.4) (layers Top Bottom) (net 1))
+  (via (at 145.7601 113.26825) (size 0.8) (drill 0.4) (layers Top Bottom) (net 1))
+  (via (at 142.6869 121.348625) (size 0.8) (drill 0.4) (layers Top Bottom) (net 1))
+  (via (at 145.7601 121.348625) (size 0.8) (drill 0.4) (layers Top Bottom) (net 1))
+  (via (at 142.6869 129.429) (size 0.8) (drill 0.4) (layers Top Bottom) (net 1))
+  (via (at 145.7601 129.429) (size 0.8) (drill 0.4) (layers Top Bottom) (net 1))
   (via (at 152.167166 111.009499) (size 0.8) (drill 0.4) (layers Top Bottom) (net 1))
   (via (at 154.283832 111.009499) (size 0.8) (drill 0.4) (layers Top Bottom) (net 1))
@@
   (segment (start 160.38534 103.80684) (end 160.38534 102.91784) (width 0.254) (layer Top) (net 1))
   (segment (start 161.8911 105.3126) (end 160.38534 103.80684) (width 0.254) (layer Top) (net 1))
-  (via (at 88.5529 98.1075) (size 0.8) (drill 0.4) (layers Top Bottom) (net 1))
-  (via (at 98.4797 98.1075) (size 0.8) (drill 0.4) (layers Top Bottom) (net 1))
-  (via (at 118.3333 98.1075) (size 0.8) (drill 0.4) (layers Top Bottom) (net 1))
-  (via (at 128.2601 98.1075) (size 0.8) (drill 0.4) (layers Top Bottom) (net 1))
-  (via (at 108.4065 98.1075) (size 0.8) (drill 0.4) (layers Top Bottom) (net 1))
-  (via (at 138.1869 98.1075) (size 0.8) (drill 0.4) (layers Top Bottom) (net 1))
+  (via (at 85.742988 97.1075) (size 0.8) (drill 0.4) (layers Top Bottom) (net 1))
+  (via (at 92.860976 97.1075) (size 0.8) (drill 0.4) (layers Top Bottom) (net 1))
+  (via (at 121.332928 97.1075) (size 0.8) (drill 0.4) (layers Top Bottom) (net 1))
+  (via (at 145.7601 97.1075) (size 0.8) (drill 0.4) (layers Top Bottom) (net 1))
+  (via (at 107.096952 97.1075) (size 0.8) (drill 0.4) (layers Top Bottom) (net 1))
+  (via (at 142.6869 97.1075) (size 0.8) (drill 0.4) (layers Top Bottom) (net 1))
   (segment (start 158.0136 123.2611) (end 160.5536 123.2611) (width 0.508) (layer Top) (net 2))
   (segment (start 161.6586 129.6296) (end 161.6586 125.3211) (width 0.508) (layer Top) (net 2))
@@
     (polygon
       (pts
-        (xy 218 137.5) (xy 79 137.5) (xy 79 72.5) (xy 218 72.5)
+        (xy 218 137.5) (xy 140.5 137.5) (xy 140.5 101) (xy 79 101) (xy 79 72.5)
+        (xy 218 72.5)
       )
     )
@@
     (polygon
       (pts
-        (xy 218 137.5) (xy 79 137.5) (xy 79 72.5) (xy 218 72.5)
+        (xy 218 137.5) (xy 140.5 137.5) (xy 140.5 101) (xy 79 101) (xy 79 72.5)
+        (xy 218 72.5)
       )
     )
