File: kicad/M17_soundcard.sch (KiCad schematic (older format))
At the start: 57 parts, among them CN1 USBMINIB, IC1 7404D, IC2 74HCT4017D, IC3 74HCT4017D, IC4 74HCT4046D, U1 CM6206, X1 10M_REF, X2 12MHz, X3 INP_A, X4 INP_B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

Commit message: Updated the values of some components, re-generated the schematic PDF file
Parts:
- C22: value TBF -> 22nF
- C23: value TBF -> 100nF
- R10: value TBF -> 56k
- R11, R12: value 1k -> 47k
- R9: value TBF -> 1k
Other:
- moved on the sheet: C10, C16, C17, C18, C19, C20, C21, C24, C25, C26, C27, C4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

Commit message: Changed value of R10 too 100 ohm
Parts:
- R10: value 56k -> 100R
Changed lines of the file:
@@
 P 8550 3650
 F 0 "R10" H 8400 3709 59  0000 L BNN
-F 1 "56k" H 8400 3520 59  0000 L BNN
+F 1 "100R" H 8400 3520 59  0000 L BNN
 F 2 "M17_soundcard:R0805" H 8550 3650 50  0001 C CNN
 F 3 "" H 8550 3650 50  0001 C CNN

Commit message: Update components' values for PLL filter
Parts:
- C22: value 22nF -> 15nF
- C23: value 100nF -> 68nF
- R10: value 100R -> 56k
Changed lines of the file:
@@
 P 8550 3650
 F 0 "R10" H 8400 3709 59  0000 L BNN
-F 1 "100R" H 8400 3520 59  0000 L BNN
+F 1 "56k" H 8400 3520 59  0000 L BNN
 F 2 "M17_soundcard:R0805" H 8550 3650 50  0001 C CNN
 F 3 "" H 8550 3650 50  0001 C CNN
@@
 P 8050 3850
 F 0 "C22" H 8125 3675 59  0000 L BNN
-F 1 "22nF" H 8125 3575 59  0000 L BNN
+F 1 "15nF" H 8125 3575 59  0000 L BNN
 F 2 "M17_soundcard:C0805" H 8050 3850 50  0001 C CNN
 F 3 "" H 8050 3850 50  0001 C CNN
@@
 P 8550 4150
 F 0 "C23" H 8275 4050 59  0000 L BNN
-F 1 "100nF" H 8175 4150 59  0000 L BNN
+F 1 "68nF" H 8175 4150 59  0000 L BNN
 F 2 "M17_soundcard:C0805" H 8550 4150 50  0001 C CNN
 F 3 "" H 8550 4150 50  0001 C CNN
